File: Hardware/PA.kicad_sch (KiCad schematic)
At the start: 57 parts, among them J3 BNC, J6 +12V, Q3 IRLML2060, T1 1:1 FT37-43, U10 TPS5430DDA, U4 LM7805_TO220, U6 INA219AxD, U8 74HC14

Commit message: Jul 1, 2024, 1:31 PM
Parts:
- renumbered C32 to C39, C32 to C6, R10 to R20, R10 to R21
