File: Hardware/Receiver.kicad_sch (KiCad schematic)
At the start: 77 parts, among them J2 BNC, J4 Audio Out to Soundcard, Q3 IRLML2060, U1 PCM1808PWR, U2 SN74CBT3253CPWR, U3 OPA1612AxD, U5 MS5351M, U7 LM2937xS, Y2 X322525MSB4SI

Commit message: Jul 1, 2024, 1:31 PM
Parts:
- renumbered C46 to C10, C46 to C14, C46 to C15, C46 to C19, C24 to C21, C24 to C22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
