File: Hardware/SDR-TRX.kicad_pcb (KiCad board)
At the start: 4 copper layers, 100 x 100 mm, 141 parts, among them J1 Debug Connector, J2 BNC, J3 BNC, J4 Audio Out to Soundcard, J6 +12V, Q2 IRLML2060, Q3 IRLML2060, SW2 RESET, T1 1:1 FT37-43, U1 PCM1808PWR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

Commit message: Jul 1, 2024, 1:31 PM
Other:
- board text added: "Put the MS5351M as close to the mixer as possible with carefully chosen equal lengths for the I_LO and Q_LO."
