File: Hardware/SDR-TRX.kicad_sch (KiCad schematic)
At the start: 7 parts, among them J1 Debug Connector, SW1 RESET, U11 CJ432, U9 Pico

Commit message: May 19, 2024, 1:57 PM
Other:
- note added: "For some reason we need a small load (33 pF works or a scope probe) between LRCK and GND."
Changed lines of the file:
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@@
     (effects (font (size 2.54 2.54) (thickness 0.508) bold) (justify left bottom))
+  )
+  (text "For some reason we need a small load (33 pF works or a scope probe)\nbetween LRCK and GND."
+    (at 52.07 111.76 0)
+    (effects (font (size 1.27 1.27)) (justify left bottom))
   )
   (text "There is a Schottky diode\npreventing backfeeding the\ncomputer USB port."
